File: Latex-Documents/Mid-Project-Presentation/Circuits/Circuits.kicad_sch (KiCad schematic)
At the start: 13 parts, among them Q1 BFP520/INF, Q2 NPN, Q3 NPN

Commit message: updated ppt
Parts:
- added C (x2): ~, symbol Device:C
- added L_p: ~, symbol Device:L
- added R_L, r_pi: ~, symbol Device:R
- added g_mv_pi, i_in: ~, symbol Simulation_SPICE:IAM
Connections:
- net GND: now also C.2, L_p.2, R_L.2, i_in.1, r_pi.1
- new net: C.1, C.2, g_mv_pi.2, i_in.2, r_pi.2
- new net: C.1, L_p.1, R_L.1, g_mv_pi.1
Other:
- note added: "v_out"
- note added: "v_pi"

Commit message: changes
Parts:
- added C1, C2: 3.3p, symbol Device:C
- added CCc: 1m, symbol Device:C
- added C_ld: 0.208424p, symbol Device:C
- added C_src: 2.02955f, symbol Device:C
- added L_ld: 10.4421n, symbol Device:L
- added L_src: 2.03361n, symbol Device:L
- added Lp: 1n, symbol Device:L
- added Q1: BFP520/INF, symbol Simulation_SPICE:NPN
- added Q2, Q3: NPN, symbol Simulation_SPICE:NPN
- added RL: 50, symbol Device:R
- added Ri: 4.5k, symbol Device:R
- C1, C2: value 3p -> 3.3p
- Ri: value 9.3k -> 4.5k
Connections:
- net GND: now also C2.2, C_src.2, L_ld.2, Q1.2 (B), RL.1
- net VCC(5V) renamed VCC(8V)
- net VCC(8V): now also Lp.1, Ri.1
- net VEE(-5V) renamed VEE(-8V)
- net VEE(-8V): now also Q2.3 (E), Q3.3 (E)
- new net: Q2.2 (B), Q3.1 (C), Q3.2 (B), Ri.2
- new net: C1.1, CCc.1, Lp.2, Q1.1 (C)
- new net: C1.2, C2.1, Q1.3 (E), Q2.1 (C)
- new net: C_ld.2, RL.2
- new net: CCc.2, L_src.1
- new net: C_ld.1, C_src.1, L_ld.1, L_src.2
Other:
- moved on the sheet: C, C_ld, C_src, L_ld, L_p, L_src, R_L, g_mv_pi, i_in, r_pi
